Commit message: gripper robot

File: description/robot.urdf.xacro (robot description, xacro)
@@ -1,4 +1,6 @@
 <?xml version="1.0"?>
 <robot xmlns:xacro="http://www.ros.org/wiki/xacro" name="robot">
-    <xacro:include filename="robot_core.xacro" />
+    <xacro:include filename="example_robot.urdf.xacro" />
+    <!-- <xacro:include filename="robot_core.xacro" /> -->
+    <!-- <xacro:include filename="gazebo_control.xacro" /> -->
 </robot>

File: description/robot_core.xacro (robot description, xacro)
@@ -24,21 +24,24 @@
     </joint>
     <link name="chassis">
-    <visual>
-        <origin xyz="0.15 0 0.075" />
-        <geometry>
-            <box size="0.3 0.3 0.15" />
-        </geometry>
-        <material name="white" />
-    </visual>
-    <collision>
-        <origin xyz="0.15 0 0.075" />
-        <geometry>
-            <box size="0.3 0.3 0.15" />
-        </geometry>
-    </collision>
-    <xacro:inertial_box mass="0.5" x="0.3" y="0.3" z="0.15">
-        <origin xyz="0.15 0 0.075" rpy="0 0 0" />
-    </xacro:inertial_box>
+        <visual>
+            <origin xyz="0.15 0 0.075" />
+            <geometry>
+                <box size="0.3 0.3 0.15" />
+            </geometry>
+            <material name="white" />
+        </visual>
+        <collision>
+            <origin xyz="0.15 0 0.075" />
+            <geometry>
+                <box size="0.3 0.3 0.15" />
+            </geometry>
+        </collision>
+        <xacro:inertial_box mass="0.5" x="0.3" y="0.3" z="0.15">
+            <origin xyz="0.15 0 0.075" rpy="0 0 0" />
+        </xacro:inertial_box>
     </link>
+    <gazebo reference="chassis">
+        <material>Gazebo/White</material>
+    </gazebo>
     <!-- Left Wheel Link(50mm radius ) -->
     <joint name="left_wheel_joint" type="continuous">
@@ -54,19 +57,22 @@
     </joint>
     <link name="left_wheel">
-    <visual>
-        <geometry>
-            <cylinder radius="0.05" length="0.04" />
-        </geometry>
-        <material name="blue" />
-    </visual>
-    <collision>
-        <geometry>
-            <cylinder radius="0.05" length="0.04" />
-        </geometry>
-    </collision>
-    <xacro:inertial_cylinder mass="0.1" length="0.04" radius="0.05">
-        <origin xyz="0 0 0" rpy="0 0 0" />
-    </xacro:inertial_cylinder>
+        <visual>
+            <geometry>
+                <cylinder radius="0.05" length="0.04" />
+            </geometry>
+            <material name="blue" />
+        </visual>
+        <collision>
+            <geometry>
+                <cylinder radius="0.05" length="0.04" />
+            </geometry>
+        </collision>
+        <xacro:inertial_cylinder mass="0.1" length="0.04" radius="0.05">
+            <origin xyz="0 0 0" rpy="0 0 0" />
+        </xacro:inertial_cylinder>
     </link>
+    <gazebo reference="left_wheel">
+        <material>Gazebo/Blue</material>
+    </gazebo>
     <!-- Right Wheel Link(50mm radius ) -->
     <joint name="right_wheel_joint" type="continuous">
@@ -77,19 +83,22 @@
     </joint>
     <link name="right_wheel">
-    <visual>
-        <geometry>
-            <cylinder radius="0.05" length="0.04" />
-        </geometry>
-        <material name="blue" />
-    </visual>
-    <collision>
-        <geometry>
-            <cylinder radius="0.05" length="0.04" />
-        </geometry>
-    </collision>
-    <xacro:inertial_cylinder mass="0.1" length="0.04" radius="0.05">
-        <origin xyz="0 0 0" rpy="0 0 0" />
-    </xacro:inertial_cylinder>
+        <visual>
+            <geometry>
+                <cylinder radius="0.05" length="0.04" />
+            </geometry>
+            <material name="blue" />
+        </visual>
+        <collision>
+            <geometry>
+                <cylinder radius="0.05" length="0.04" />
+            </geometry>
+        </collision>
+        <xacro:inertial_cylinder mass="0.1" length="0.04" radius="0.05">
+            <origin xyz="0 0 0" rpy="0 0 0" />
+        </xacro:inertial_cylinder>
     </link>
+    <gazebo reference="right_wheel">
+        <material>Gazebo/Blue</material>
+    </gazebo>
     <!-- Caster Wheel Link -->
     <joint name="caster_wheel_joint" type="fixed">
@@ -99,18 +108,23 @@
     </joint>
     <link name="caster_wheel">
-    <visual>
-        <geometry>
-            <sphere radius="0.05" />
-        </geometry>
-        <material name="black" />
-    </visual>
-    <collision>
-        <geometry>
-            <sphere radius="0.05" />
-        </geometry>
-    </collision>
-    <xacro_inertial_sphere mass="0.1" radius="0.05">
-        <origin xyz="0 0 0" rpy="0 0 0" />
-    </xacro_inertial_sphere>
+        <visual>
+            <geometry>
+                <sphere radius="0.05" />
+            </geometry>
+            <material name="black" />
+        </visual>
+        <collision>
+            <geometry>
+                <sphere radius="0.05" />
+            </geometry>
+        </collision>
+        <xacro_inertial_sphere mass="0.1" radius="0.05">
+            <origin xyz="0 0 0" rpy="0 0 0" />
+        </xacro_inertial_sphere>
     </link>
+    <gazebo reference="caster_wheel">
+        <material>Gazebo/Black</material>
+        <mu1 value="0.001" />
+        <mu2 value="0.001" />
+    </gazebo>
 </robot>

Commit message: lidar in ros

File: description/robot.urdf.xacro (robot description, xacro)
@@ -1,6 +1,6 @@
 <?xml version="1.0"?>
 <robot xmlns:xacro="http://www.ros.org/wiki/xacro" name="robot">
-    <xacro:include filename="example_robot.urdf.xacro" />
-    <!-- <xacro:include filename="robot_core.xacro" /> -->
-    <!-- <xacro:include filename="gazebo_control.xacro" /> -->
+    <xacro:include filename="robot_core.xacro" />
+    <xacro:include filename="gazebo_control.xacro" />
+    <xacro:include filename="lidar.xacro" />
 </robot>

File: description/robot_core.xacro (robot description, xacro)
@@ -13,4 +13,7 @@
     <material name="black">
         <color rgba="0 0 0 1" />
+    </material>
+    <material name="red">
+        <color rgba="1 0 0 1" />
     </material>
     <!-- Base Link -->
